File: hv_board/hv_board.kicad_sch (KiCad schematic)
At the start: 31 parts, among them J6 Controller board, K1 RT314A12, Q1 BSS138, Q2 BSS138, Q3 BTA16-600BWRG, U1 ECE10US12, U2 ALDP112, U3 BAT46WJ_115, U4 BAT46WJ_115, U5 H11L1, U7 MOC3021M

Commit message: New gerber files
Parts:
- R8: value 86.6 -> 100
Changed lines of the file:
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@@
 			)
 		)
-		(property "Value" "86.6"
+		(property "Value" "100"
 			(at 246.38 133.35 90)
 			(effects
