File: hv_board/hv_board.kicad_pcb (KiCad board)
At the start: 2 copper layers, 69 x 54 mm, 33 parts, among them J6 Controller board, K1 RT314A12, Q1 BSS138, Q2 BSS138, Q3 BTA16-600BWRG, U1 ECE10US12, U2 ALDP112, U3 BAT46WJ_115, U4 BAT46WJ_115, U5 H11L1, U7 MOC3021M

Commit message: New gerber files
Parts:
- R8: value 86.6 -> 100
Changed lines of the file:
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@@
 			)
 		)
-		(property "Value" "86.6"
+		(property "Value" "100"
 			(at 0 1.65 90)
 			(layer "F.Fab")
@@
 			(hide yes)
 			(effects
+				(font
+					(size 1.27 1.27)
+					(thickness 0.15)
+				)
+			)
+		)
+		(property "LCSC" "C17408"
+			(at 0 0 0)
+			(layer "F.SilkS")
+			(hide yes)
+			(effects

Commit message: Many fixes
Other:
- board text added: "MaraXEvolution HV Rev1.0a"
Changed lines of the file:
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@@
 		(layer "Edge.Cuts")
+	)
+	(gr_text "MaraXEvolution HV Rev1.0a"
+		(at 141.8 67.6 0)
+		(layer "F.SilkS")
+		(effects
+			(font
+				(size 1 1)
+				(thickness 0.1)
+			)
+			(justify left bottom)
+		)
 	)
 	(via
@@
 	)
 	(via
-		(at 164 68)
+		(at 164 66.2)
 		(size 0.6)
 		(drill 0.3)
@@
 		(start 157 93.5)
 		(end 157 89)
-		(width 1.2)
+		(width 0.6)
 		(layer "F.Cu")
 		(net 12)
@@
 	(via
 		(at 157 89)
-		(size 1.2)
-		(drill 0.8)
+		(size 0.6)
+		(drill 0.3)
 		(layers "F.Cu" "B.Cu")
 		(net 12)
@@
 		(start 160.25 85.75)
 		(end 157 89)
-		(width 1.2)
+		(width 0.6)
 		(layer "B.Cu")
 		(net 12)
 	)
 	(segment
+		(start 177.32 85.75)
+		(end 163.25 85.75)
+		(width 0.6)
+		(layer "B.Cu")
+		(net 12)
+	)
+	(segment
 		(start 179.545 87.975)
-		(end 178.975 87.975)
-		(width 1.2)
-		(layer "B.Cu")
-		(net 12)
-	)
-	(segment
-		(start 176.75 85.75)
-		(end 163.25 85.75)
-		(width 1.2)
+		(end 177.32 85.75)
+		(width 0.6)
 		(layer "B.Cu")
 		(net 12)
@@
 		(start 163.25 85.75)
 		(end 160.25 85.75)
-		(width 1.2)
-		(layer "B.Cu")
-		(net 12)
-	)
-	(segment
-		(start 178.975 87.975)
-		(end 177 86)
-		(width 1.2)
-		(layer "B.Cu")
-		(net 12)
-	)
-	(segment
-		(start 177 86)
-		(end 176.75 85.75)
-		(width 1.2)
+		(width 0.6)
 		(layer "B.Cu")
 		(net 12)
@@
 		(start 182 94)
 		(end 182 93.5)
-		(width 1.2)
+		(width 0.6)
 		(layer "B.Cu")
 		(net 13)
@@
 		(start 173.5 67)
 		(end 178.5 67)
-		(width 1.2)
+		(width 0.6)
 		(layer "B.Cu")
 		(net 13)
@@
 		(start 182 70.5)
 		(end 182 78)
-		(width 1.2)
+		(width 0.6)
 		(layer "B.Cu")
 		(net 13)
@@
 		(start 182 78)
 		(end 182 93.5)
-		(width 1.2)
+		(width 0.6)
 		(layer "B.Cu")
 		(net 13)
@@
 		(start 174.465 93.055)
 		(end 176.91 95.5)
-		(width 1.2)
+		(width 0.6)
 		(layer "B.Cu")
 		(net 13)
@@
 		(start 178.5 67)
 		(end 182 70.5)
-		(width 1.2)
+		(width 0.6)
 		(layer "B.Cu")
 		(net 13)
@@
 		(start 180.5 95.5)
 		(end 182 94)
-		(width 1.2)
+		(width 0.6)
 		(layer "B.Cu")
 		(net 13)
@@
 		(start 176.91 95.5)
 		(end 180.5 95.5)
-		(width 1.2)
+		(width 0.6)
 		(layer "B.Cu")
 		(net 13)
@@
 		(start 149 74)
 		(end 145.011 77.989)
-		(width 0.4)
+		(width 0.6)
 		(layer "F.Cu")
 		(net 19)
@@
 		(start 145.011 77.989)
 		(end 145.011 87.511)
-		(width 0.4)
+		(width 0.6)
 		(layer "F.Cu")
 		(net 19)
@@
 		(start 152.5 91)
 		(end 155 93.5)
-		(width 0.4)
+		(width 0.6)
 		(layer "F.Cu")
 		(net 19)
@@
 		(start 148.5 91)
 		(end 152.5 91)
-		(width 0.4)
+		(width 0.6)
 		(layer "F.Cu")
 		(net 19)
@@
 		(start 145.011 87.511)
 		(end 148.5 91)
-		(width 0.4)
+		(width 0.6)
 		(layer "F.Cu")
 		(net 19)
@@
 		(start 163.001 76.501)
 		(end 158 71.5)
-		(width 0.4)
+		(width 0.6)
 		(layer "B.Cu")
 		(net 19)
@@
 		(start 165.499 76.501)
 		(end 163.001 76.501)
-		(width 0.4)
+		(width 0.6)
 		(layer "B.Cu")
 		(net 19)
@@
 		(start 165.499 76.501)
 		(end 172.46 69.54)
-		(width 0.4)
+		(width 0.6)
 		(layer "B.Cu")
 		(net 19)
@@
 		(start 151.5 71.5)
 		(end 149 74)
-		(width 0.4)
+		(width 0.6)
 		(layer "B.Cu")
 		(net 19)
@@
 		(start 172.46 69.54)
 		(end 173.61 69.54)
-		(width 0.4)
+		(width 0.6)
 		(layer "B.Cu")
 		(net 19)
@@
 		(start 158 71.5)
 		(end 151.5 71.5)
-		(width 0.4)
+		(width 0.6)
 		(layer "B.Cu")
 		(net 19)
@@
 	)
 	(segment
-		(start 163.233607 67.633607)
-		(end 158.4 62.8)
-		(width 0.6)
-		(layer "B.Cu")
-		(net 21)
-	)
-	(segment
-		(start 163.199 68.331786)
-		(end 163.199 67.668214)
-		(width 0.6)
-		(layer "B.Cu")
-		(net 21)
-	)
-	(segment
-		(start 163.199 67.668214)
-		(end 163.233607 67.633607)
-		(width 0.6)
-		(layer "B.Cu")
-		(net 21)
-	)
-	(segment
-		(start 163.668214 68.801)
-		(end 163.199 68.331786)
-		(width 0.6)
-		(layer "B.Cu")
-		(net 21)
-	)
-	(segment
-		(start 165.14 69.54)
-		(end 164.366393 68.766393)
-		(width 0.6)
-		(layer "B.Cu")
-		(net 21)
-	)
-	(segment
-		(start 164.331786 68.801)
-		(end 163.668214 68.801)
+		(start 165.99 69.54)
+		(end 165.14 69.54)
 		(width 0.6)
 		(layer "B.Cu")
@@
 	)
 	(segment
-		(start 165.99 69.54)
-		(end 165.14 69.54)
-		(width 0.6)
-		(layer "B.Cu")
-		(net 21)
-	)
-	(segment
-		(start 164.366393 68.766393)
-		(end 164.331786 68.801)
+		(start 165.14 69.54)
+		(end 158.4 62.8)
 		(width 0.6)
 		(layer "B.Cu")
@@
 		(layer "B.Cu")
 		(net 29)
-	)
-	(zone
-		(net 19)
-		(net_name "Net-(R7-Pad2)")
-		(layer "F.Cu")
-		(name "$teardrop_padvia$")
-		(hatch none 0.1)
-		(priority 30000)
-		(attr
-			(teardrop
-				(type padvia)
-			)
-		)
-		(connect_pads yes
-			(clearance 0)
-		)
-		(min_thickness 0.0254)
-		(filled_areas_thickness no)
-		(fill yes
-			(thermal_gap 0.5)
-			(thermal_bridge_width 0.5)
-			(island_removal_mode 1)
-			(island_area_min 10)
-		)
-		(polygon
-			(pts
-				(xy 148.438391 74.278766) (xy 148.721234 74.561609) (xy 149.166671 74.249441) (xy 149.000707 73.999293)
-				(xy 148.750559 73.833329)
-			)
-		)
 	)
 	(zone
@@
 			)
 		)
-	)
-	(zone
-		(net 19)
-		(net_name "Net-(R7-Pad2)")
-		(layer "B.Cu")
-		(name "$teardrop_padvia$")
-		(hatch none 0.1)
-		(priority 30000)
-		(attr
-			(teardrop
-				(type padvia)
-			)
-		)
-		(connect_pads yes
-			(clearance 0)
-		)
-		(min_thickness 0.0254)
-		(filled_areas_thickness no)
-		(fill yes
-			(thermal_gap 0.5)
-			(thermal_bridge_width 0.5)
-			(island_removal_mode 1)
-			(island_area_min 10)
-		)
-		(polygon
-			(pts
-				(xy 149.561609 73.721234) (xy 149.278766 73.438391) (xy 148.833329 73.750559) (xy 148.999293 74.000707)
-				(xy 149.249441 74.166671)
-			)
-		)
