File: controller_board/controller_board.kicad_pcb (KiCad board)
At the start: 2 copper layers, 69 x 54 mm, 75 parts, among them CN1 Boiler fill sensor, CN2 Water level detector, CN3 Sensor steam boiler, CN4 Sensor brew boiler, CN5 Heater SSR Relay, CN6 MISC LEDS, CN7 Brew switch, IC1 AQV212, IC2 LM4050AEM3-3.0+T, J2 HV Board, J4 705530002, J5 705530041, Q1 BSS138, Q2 BSS138, Q3 BSS138, Q4 BSS138, U1 ADS1115IDGS, U2 LM1830N, U3 IE092503-1

Commit message: Many fixes
Connections:
- R39 pad 2: D8 -> A2
Routing:
- net A2: track 0.00 -> 35.7 mm, vias 0 -> 2
- net D8: track 12.4 -> 0.00 mm
Other:
- board text added: "MaraXEvolution Controller Rev1.0a"
Changed lines of the file:
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@@
 		(tags "resistor handsolder")
 		(property "Reference" "R11"
-			(at 0 -1.65 270)
+			(at 0 1.8 270)
 			(layer "F.SilkS")
 			(effects
@@
 		(tags "resistor handsolder")
 		(property "Reference" "R22"
-			(at 0 -1.65 270)
+			(at -0.2 1.6 270)
 			(layer "F.SilkS")
 			(effects
@@
 		(tags "resistor handsolder")
 		(property "Reference" "R6"
-			(at 0 -1.65 270)
+			(at 0 1.6 270)
 			(layer "F.SilkS")
 			(effects
@@
 			)
 		)
-		(property "LCSC" ""
-			(at 0 0 0)
-			(layer "F.SilkS")
-			(hide yes)
-			(effects
-				(font
-					(size 1.27 1.27)
-					(thickness 0.15)
-				)
-			)
-		)
 		(sheetname "/")
 		(sheetfile "controller_board.kicad_sch")
@@
 		(tags "resistor handsolder")
 		(property "Reference" "R18"
-			(at 0 -1.65 270)
+			(at 0 1.8 270)
 			(layer "F.SilkS")
 			(effects
@@
 			)
 		)
-		(property "LCSC" ""
-			(at 0 0 0)
-			(layer "F.SilkS")
-			(hide yes)
-			(effects
-				(font
-					(size 1.27 1.27)
-					(thickness 0.15)
-				)
-			)
-		)
 		(sheetname "/")
 		(sheetfile "controller_board.kicad_sch")
@@
 		(tags "VSSOP SO")
 		(property "Reference" "U1"
-			(at 0 -2.45 180)
+			(at 0 0 180)
 			(layer "F.SilkS")
 			(effects
@@
 			(layers "F.Cu" "F.Mask" "F.Paste")
 			(roundrect_rratio 0.208333)
-			(net 35 "D8")
+			(net 39 "A2")
 			(pintype "passive")
 		)
@@
 		(tags "resistor handsolder")
 		(property "Reference" "R31"
-			(at 0 -1.65 0)
+			(at 0 -1.6 0)
 			(layer "F.SilkS")
 			(effects
@@
 		(layer "Edge.Cuts")
 	)
+	(gr_text "MaraXEvolution Controller Rev1.0a"
+		(at 81.6 92.4 0)
+		(layer "F.SilkS")
+		(effects
+			(font
+				(size 1 1)
+				(thickness 0.1)
+			)
+			(justify left bottom)
+		)
+	)
 	(gr_text "5"
 		(at 116.6 71.039999 180)
@@
 	)
 	(segment
-		(start 83.74 86)
-		(end 86 88.26)
-		(width 0.4)
-		(layer "F.Cu")
-		(net 35)
-	)
-	(segment
-		(start 75.2 84.4)
-		(end 77.6 84.4)
-		(width 0.4)
-		(layer "F.Cu")
-		(net 35)
-	)
-	(segment
-		(start 77.6 84.4)
-		(end 79.2 86)
-		(width 0.4)
-		(layer "F.Cu")
-		(net 35)
-	)
-	(segment
-		(start 79.2 86)
-		(end 83.74 86)
-		(width 0.4)
-		(layer "F.Cu")
-		(net 35)
-	)
-	(segment
 		(start 111.575 76.2)
 		(end 111.775 76)
@@
 	)
 	(segment
+		(start 88.54 103.5)
+		(end 88.54 98.94)
+		(width 0.4)
+		(layer "F.Cu")
+		(net 39)
+	)
+	(segment
+		(start 75.2 84.4)
+		(end 77.6 84.4)
+		(width 0.4)
+		(layer "F.Cu")
+		(net 39)
+	)
+	(segment
+		(start 88.54 98.94)
+		(end 87.4 97.8)
+		(width 0.4)
+		(layer "F.Cu")
+		(net 39)
+	)
+	(via
+		(at 87.4 97.8)
+		(size 0.6)
+		(drill 0.3)
+		(layers "F.Cu" "B.Cu")
+		(net 39)
+	)
+	(via
+		(at 77.6 84.4)
+		(size 0.6)
+		(drill 0.3)
+		(layers "F.Cu" "B.Cu")
+		(net 39)
+	)
+	(segment
+		(start 74 85.6)
+		(end 75.2 84.4)
+		(width 0.4)
+		(layer "B.Cu")
+		(net 39)
+	)
+	(segment
+		(start 72.4 87.2)
+		(end 74 85.6)
+		(width 0.4)
+		(layer "B.Cu")
+		(net 39)
+	)
+	(segment
+		(start 80.6 97.8)
+		(end 72.4 89.6)
+		(width 0.4)
+		(layer "B.Cu")
+		(net 39)
+	)
+	(segment
+		(start 72.4 89.6)
+		(end 72.4 87.2)
+		(width 0.4)
+		(layer "B.Cu")
+		(net 39)
+	)
+	(segment
+		(start 75.2 84.4)
+		(end 77.6 84.4)
+		(width 0.4)
+		(layer "B.Cu")
+		(net 39)
+	)
+	(segment
+		(start 87.4 97.8)
+		(end 80.6 97.8)
+		(width 0.4)
+		(layer "B.Cu")
+		(net 39)
+	)
+	(segment
