File: controller_board/controller_board.kicad_sch (KiCad schematic)
At the start: 73 parts, among them CN1 Boiler fill sensor, CN2 Water level detector, CN3 Sensor steam boiler, CN4 Sensor brew boiler, CN5 Heater SSR Relay, CN6 MISC LEDS, CN7 Brew switch, IC1 AQV212, IC2 LM4050AEM3-3.0+T, J2 HV Board, J4 705530002, J5 705530041, Q1 BSS138, Q2 BSS138, Q3 BSS138, Q4 BSS138, U1 ADS1115IDGS, U2 LM1830N, U3 IE092503-1

Commit message: Many fixes
Connections:
- net A2: now also R39.2
- net D8: no longer R39.2
